File: chufe/hardware/chufe-v-0-rev-a/chufe-v-0-rev-a.kicad_pcb (KiCad board)
At the start: 2 copper layers, 50 x 65 mm, 23 parts, among them J1 Conn_02x08_Odd_Even, J2 Conn_01x04_Pin, J3 Barrel_Jack_Switch, Q1 AO3401A, U1 URA2412YMD-20WR3_C5369773, U2 L7805

Commit message: agregar chufebu and chufe
Other:
- board text added: "2026-10"
- board text added: "chufe"
- board text added: "rev a"
- board text added: "v0"
